Commit message: Update URDF, add lidar description, add collisions

File: src/capo_description/src/description/capo_description.urdf (robot description, URDF)
Before this commit: robot capo, 2 links, 1 joints
Links:
- added link lidar_link; collision cylinder length=0.07 radius=0.0235; visual cylinder length=0.07 radius=0.0235
- link base_link: geometry collision box size=${base_length} ${base_width} ${base_height}; visual box size=${base_length} ${base_width} ${base_height}
Joints:
- added joint lidar_joint: type fixed, parent base_link, child lidar_link, origin xyz=1.85 0 ${base_height/2+0.035} rpy=0 0 0

Commit message: Comment out an unnecessary node and fix typos

File: src/capo_description/src/description/capo_description.urdf (robot description, URDF)
Before this commit: robot capo, 3 links, 2 joints
Joints:
- joint lidar_joint: origin xyz=1.85 0 ${base_height/2+0.035} rpy=0 0 0 -> xyz=0.0185 0 ${base_height/2} rpy=0 0 0

Commit message: Adjust laser scaner position

File: src/capo_description/src/description/capo_description.urdf (robot description, URDF)
Before this commit: robot capo, 3 links, 2 joints
Joints:
- joint lidar_joint: origin xyz=0.0185 0 ${base_height/2} rpy=0 0 0 -> xyz=0.0185 0 ${base_height/2+0.035} rpy=0 0 0
